File: hw/PCB/FOD.sch (KiCad schematic (older format))
At the start: 8 parts, among them J2 Programmer, U1 SAMD21G, U2 Payload, Y1 32.768kHz

Commit message: Finished preliminary design phase for the version 2.0.
Parts:
- removed J2: Programmer, Connector_PinHeader_2.54mm:PinHeader_1x04_P2.54mm_Vertical, symbol Connector:Conn_01x04_Male
- removed JP1: Jumper_NC_Dual, Connector_PinHeader_2.54mm:PinHeader_1x03_P2.54mm_Vertical, symbol Device:Jumper_NC_Dual
- removed R1: 1k, Resistor_SMD:R_0603_1608Metric_Pad1.05x0.95mm_HandSolder, symbol Device:R
- removed U1: SAMD21G, Package_QFP:TQFP-48_7x7mm_P0.5mm, symbol Arduino:SAMD21G
- removed U2: Payload, Payload:FOD, symbol Payload:Payload
- added U0: Payload, Payload:FOD, symbol Payload:Payload
- added U1: SAMD21E, Package_QFP:TQFP-32_7x7mm_P0.8mm, symbol Arduino:SAMD21E
Connections:
- net 3V3: now also U1.30 (VDDIN)
- net DPL_EN: now also U1.14 (PA11/0)
- net GND: now also U0.81 (29-GND), U0.82 (GND-30), U0.84 (GND-32), U1.10 (GND), U1.28 (GND)
- net MISO: now also U1.20 (PA19/12/MISO)
- net MOSI: now also U1.17 (PA16/11/MOSI)
- net RESET: now also U1.26 (RESET)
- net SCK: now also U1.18 (PA17/13/SCK)
- net SCL: now also U0.11 (11-I2C2_SCL), U1.22 (PA23/SCL)
- net SDA: now also U0.9 (09-I2C2_SDA), U1.21 (PA22/SDA)
- net SWCLK: now also U1.31 (PA30/SWCLK)
- net SWDIO: now also U1.32 (PA31/SWDIO)
- net TRX_INT: now also U1.15 (PA14/2)
- net TRX_NSS: now also U1.19 (PA18/10/SS)
- net TRX_RST: now also U1.16 (PA15/5)
- net USB_ID: now also U1.27 (PA28_USB_ID)
- net USB_N: now also U1.23 (PA24_USB_DM)
- net USB_P: now also U1.24 (PA25_USB_DP)
- net VDDANA: now also U1.9 (VDDANA)
- net VDDCORE: now also U1.29 (VDDCORE)
- net VIN: now also U0.50 (OUT5_5V0-50)
- net XIN32: now also U1.1 (PA00/XIN32)
- net XOUT32: now also U1.2 (PA01/XOUT32)
- new net DPL_STA: U1.13 (PA10/1)
- no-connect marks 0 -> 9
