File: hw/PCB/FOD.sch (KiCad schematic (older format))
At the start: 6 parts, among them J2 I2C, J3 I2C, U1 SAMD21G, Y1 32.768kHz

Commit message: Separated the VIN power line into two independent power lines (VAUX and VAUX2). This is done to add compatibility with other CubeSats standards. Added the option to bridge those lines with a zero Ohm resistor.
Parts:
- added R8: 0, Resistor_SMD:R_0603_1608Metric_Pad1.05x0.95mm_HandSolder, symbol Device:R
Connections:
- net labels added: VAUX, VAUX2
- net labels removed: VIN
- wire segments 97 -> 99
Changed lines of the file:
@@
 	7650 3600 7900 3600
 Wire Wire Line
-	7650 3700 7900 3700
-Wire Wire Line
-	7650 3800 7900 3800
+	7650 3700 8100 3700
+Wire Wire Line
+	7650 3800 7950 3800
+Wire Wire Line
+	7950 3800 7950 4000
+Wire Wire Line
+	7950 4000 8100 4000
 Wire Wire Line
 	8550 3300 8300 3300
@@
 MISO
 Text Label 6300 4400 0    50   ~ 0
-VIN
+VAUX
 Text Label 6300 4500 0    50   ~ 0
 3V3
@@
 GND
 Text Label 7900 3700 2    50   ~ 0
-VIN
+VAUX2
 Text Label 7900 3800 2    50   ~ 0
-VIN
+VAUX
 Text Label 7900 4400 2    50   ~ 0
 DPL_STA1
@@
 GND
 Text Label 8300 3700 0    50   ~ 0
-VIN
+VAUX2
 Text Label 8300 3800 0    50   ~ 0
-VIN
+VAUX
 $Comp
 L power:GND #PWR0104
@@
 	1    0    0    -1
 $EndComp
+$Comp
+L Device:R R8
+U 1 1 5E8670A2
+P 8100 3850
+F 0 "R8" H 8170 3805 50  0000 L CNN
+F 1 "0" H 8170 3895 50  0000 L CNN
+F 2 "Resistor_SMD:R_0603_1608Metric_Pad1.05x0.95mm_HandSolder" V 8030 3850 50  0001 C CNN
+F 3 "~" H 8100 3850 50  0001 C CNN
+	1    8100 3850
+	1    0    0    -1
+$EndComp
