File: hw/PCB/dpl.sch (KiCad schematic (older format))
At the start: 5 parts, among them J3 Nichrome, Q1 PMV16XNR, U4 AV4524

Commit message: Fixed a small issue about the pin assignation of the deployment sensor. Change the position of some vias so that they are not too close to some tracks.
Connections:
- net 3V3: now also U4.3 (NC); no longer U4.2 (NO)
- net GND: now also U4.2 (NO); no longer U4.3 (NC)
Changed lines of the file:
@@
 Text HLabel 4950 2900 0    50   Input ~ 0
 DPL_EN
-Text HLabel 4950 3950 0    50   Input ~ 0
+Text HLabel 4950 3850 0    50   Input ~ 0
 GND
 Text HLabel 5750 2550 0    50   Input ~ 0
@@
 	5150 3750 4950 3750
 Wire Wire Line
-	5150 3950 5050 3950
-Wire Wire Line
-	4950 3850 5150 3850
-Text HLabel 4950 3850 0    50   Input ~ 0
+	4950 3850 5050 3850
+Text HLabel 4950 3950 0    50   Input ~ 0
 3V3
 $Comp
@@
 	1    0    0    -1
 $EndComp
-Wire Wire Line
-	5050 4000 5050 3950
-Connection ~ 5050 3950
-Wire Wire Line
-	5050 3950 4950 3950
 $Comp
 L Device:R R5
@@
 	1    0    0    -1
 $EndComp
+Wire Wire Line
+	4950 3950 5150 3950
+Wire Wire Line
+	5050 3850 5050 4000
+Connection ~ 5050 3850
+Wire Wire Line
+	5050 3850 5150 3850
 $EndSCHEMATC
